Commit message: Update vs060-gazebo.xacro

File: vs060_gazebo/urdf/vs060-gazebo.xacro (robot description, xacro)
@@ -146,25 +146,4 @@
     </inertial>
   </link>
-  <!-- Camera -->
-  <link name="camera_link">
-    <collision>
-      <origin xyz="0 0 0" rpy="0 0 0"/>
-      <geometry>
-	<box size="0.02 0.05 0.05"/>
-      </geometry>
-    </collision>
-    <visual>
-      <origin xyz="0 0 0" rpy="0 0 0"/>
-      <geometry>
-	<box size="0.02 0.05 0.05"/>
-      </geometry>
-      <material name="green"/>
-    </visual>
-    <inertial>
-      <mass value="1e-5" />
-      <origin xyz="0 0 0" rpy="0 0 0"/>
-      <inertia ixx="1e-6" ixy="0" ixz="0" iyy="1e-6" iyz="0" izz="1e-6" />
-    </inertial>
-  </link>
   <joint name="j1" type="revolute">
     <parent link="BASE"/>
@@ -209,9 +188,3 @@
     <limit lower="-6.2831853" upper="6.2831853" effort="28.0" velocity="3.2"/>
   </joint>
-  <joint name="camera_joint" type="fixed">
-    <axis xyz="0 0 1" />
-    <origin xyz="0 0 0" rpy="3.14 -1.57 0"/>
-    <parent link="Flange"/>
-    <child link="camera_link"/>
-  </joint>
 </robot>
